File: BM3451XXDC-T28A-Board.kicad_sch (KiCad schematic)
At the start: 84 parts, among them Q1 AO3400A, Q10 NCE3080K, Q11 NCE3080K, Q2 AO3400A, Q3 AO3400A, Q4 AO3400A, Q5 AO3400A, Q6 MMBT5401, Q7 MMBT5551, Q8 NCE3080K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

Commit message: Submit readme.md and some images
Parts:
- RSENSE1, RSENSE2: value 5m -> 0.005/3W
Changed lines of the file:
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@@
     (fill (type none))
   )
-  (rectangle (start 254.635 106.045) (end 274.955 124.46)
+  (rectangle (start 254.635 106.045) (end 274.955 120.65)
     (stroke (width 0.2) (type solid))
     (fill (type none))
@@
   )
   (symbol (lib_id "Device:R") (at 161.29 170.18 270) (unit 1)
-    (in_bom yes) (on_board yes) (dnp no) (fields_autoplaced)
-    (property "Reference" "RSENSE2" (at 154.305 168.91 90)
-      (effects (font (size 1.27 1.27)))
-    )
-    (property "Value" "5m" (at 165.735 168.91 90)
+    (in_bom yes) (on_board yes) (dnp no)
+    (property "Reference" "RSENSE2" (at 153.67 168.91 90)
+      (effects (font (size 1.27 1.27)))
+    )
+    (property "Value" "0.005/3W" (at 168.91 168.91 90)
       (effects (font (size 1.27 1.27)))
     )
@@
   )
   (symbol (lib_id "Device:R") (at 161.29 165.1 270) (unit 1)
-    (in_bom yes) (on_board yes) (dnp no) (fields_autoplaced)
-    (property "Reference" "RSENSE1" (at 154.305 163.83 90)
-      (effects (font (size 1.27 1.27)))
-    )
-    (property "Value" "5m" (at 165.735 163.83 90)
-      (effects (font (size 1.27 1.27)))
-    )
+    (in_bom yes) (on_board yes) (dnp no)
+    (property "Reference" "RSENSE1" (at 153.67 163.83 90)
+      (effects (font (size 1.27 1.27)))
+    )
+    (property "Value" "0.005/3W" (at 168.91 163.83 90)
+      (effects (font (size 1.27 1.27)))
+    )
